Commit message: test(arm): update arm urdf

File: rmcs_ws/src/arm_description/urdf/arm_description.urdf (robot description, URDF)
Before this commit: robot arm_description, 7 links, 6 joints
Links:
- link link_3: mass 1.821 -> 1.1935
- link link_4: mass 1.61 -> 1.0552
- link link_5: mass 0.624 -> 0.4090

Commit message: test(arm): continue modifying urdf to tune gravity compensation

File: rmcs_ws/src/arm_description/urdf/arm_description.urdf (robot description, URDF)
Before this commit: robot arm_description, 7 links, 6 joints
Links:
- link link_3: mass 1.1935 -> 0.7935
- link link_4: mass 1.0552 -> 0.8052
- link link_6: mass 0.77108 -> 1.0262

Commit message: fix(arm): tune urdf

File: rmcs_ws/src/arm_description/urdf/arm_description.urdf (robot description, URDF)
Before this commit: robot arm_description, 7 links, 6 joints
Links:
- link link_2: mass 0.1502 -> 0.108
- link link_3: mass 0.7935 -> 1.311
- link link_4: mass 0.8052 -> 1.159
- link link_5: mass 0.4090 -> 0.449
- link link_6: mass 1.0262 -> 0.555

Commit message: test(arm): tune urdf (final)
This should be the final urdf for 6-axis arm gravity compensation.

File: rmcs_ws/src/arm_description/urdf/arm_description.urdf (robot description, URDF)
Before this commit: robot arm_description, 7 links, 6 joints
Links:
- link link_3: mass 1.311 -> 2.65
